File: MCU_DATA_LOGGER.kicad_pcb (KiCad board)
At the start: 2 copper layers, 49.3 x 31.2 mm, 29 parts, among them J1 Conn_01x04_Male, J2 Conn_01x04_Male, J3 Conn_01x09_Male, J4 Conn_02x03_Odd_Even, U1 DS1337S+, U2 24LC1025, U3 24LC1025, U4 ATMEGA328P-AU, Y1 32.768 KHz, Y2 16 MHz

Commit message: completed 4 layer
Parts:
- moved R5 5.85 mm to (81.8, 72.1)
- moved D3 2.97 mm to (77.7, 73.9)
Routing:
- net /Vcc: track 203.0 -> 55.2 mm, vias 6 -> 9
- net GND: track 100.2 -> 40.8 mm, vias 9 -> 12
- net /SCK: track 109.7 -> 87.6 mm, vias 8 -> 5
- net Net-(C4-Pad2): track 35.1 -> 17.1 mm
- net /MISO: track 43.5 -> 28.0 mm, vias 4 -> 2
- net /SDA: track 67.0 -> 57.4 mm
- net Net-(D2-Pad1): track 11.6 -> 3.82 mm
- net /D8: track 11.9 -> 19.3 mm, vias 1 -> 0
- net Net-(C3-Pad2): track 30.2 -> 23.1 mm, vias 2 -> 3
- net /Tx: track 30.7 -> 36.0 mm, vias 1 -> 0
- net /D7: track 12.6 -> 15.9 mm, vias 1 -> 0
- net /D2: track 32.1 -> 29.5 mm
- net /RESET: track 25.4 -> 22.9 mm
- net Net-(R1-Pad2): track 9.21 -> 7.48 mm
- net Net-(D3-Pad1): track 6.61 -> 5.22 mm
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- added copper zone on In2.Cu, net /Vcc
Other:
- copper layers 2 -> 4

Commit message: Completed all + board characteristics
Other:
- board text added: "0,2000 mm / 0,0000 mm"
- board text added: "0,3000 mm"
- board text added: "4"
- board text added: "4,6900 mm"
- board text added: "49,3760 mm x 31,3420 mm"
- board text added: "BOARD CHARACTERISTICS"
- board text added: "Board Thickness:"
- board text added: "Board overall dimensions:"
- board text added: "Castellated pads:"
- board text added: "Copper Finish:"
- board text added: "Copper Layer Count:"
- board text added: "Edge card connectors:"
- board text added: "Impedance Control:"
- board text added: "Min hole diameter:"
- board text added: "Min track/spacing:"
- board text added: "No"
- board text added: "None"
- board text added: "Plated Board Edge:"
